File: ATmega32u4.sch (KiCad schematic (older format))
At the start: 27 parts, among them J1 USB_B_Mini, J2 AVR-ISP-6, U4 ATmega32U4RC-MU, Y1 16MHz

Commit message: Miscellaneous fixes
Parts:
- C16, C21: footprint Collins-FMS-3000:Perfect_0402 -> CJ4-MFD-Menu-Panel:Perfect_0402; LCSC C15525 -> (none)
- C17, C18, C19, C20, C23, C24: footprint Collins-FMS-3000:Perfect_0402 -> CJ4-MFD-Menu-Panel:Perfect_0402; LCSC C1525 -> (none)
- C22, C25: footprint Collins-FMS-3000:Perfect_0402 -> CJ4-MFD-Menu-Panel:Perfect_0402; LCSC C52923 -> (none)
- C26, C27: footprint Collins-FMS-3000:Perfect_0402 -> CJ4-MFD-Menu-Panel:Perfect_0402; LCSC C1554 -> (none)
- D1: footprint Collins-FMS-3000:LED_0603_1608Metric -> LED_SMD:LED_0805_2012Metric_Pad1.15x1.40mm_HandSolder; JLC 0603 -> (none)
- FB1: LCSC C72043 -> C1017
- J1: footprint Collins-FMS-3000:USB_B_Mini_Amphenol_UE25BE5510H -> CJ4-MFD-Menu-Panel:USB_B_Mini_Amphenol_UE25BE5510H
- R11, R15, R19, R21: footprint Collins-FMS-3000:Perfect_0402 -> CJ4-MFD-Menu-Panel:Perfect_0402
- R12, R14: footprint Collins-FMS-3000:Perfect_0402 -> CJ4-MFD-Menu-Panel:Perfect_0402; LCSC 0402 -> C25092
Connections:
- net DOWN: now also U4.37 (PF6); no longer U4.39 (PF4)
- net UP: now also U4.39 (PF4); no longer U4.37 (PF6)
Changed lines of the file:
@@
 F 0 "C16" H 892 1096 50  0000 L CNN
 F 1 "10uF" H 892 1005 50  0000 L CNN
-F 2 "Collins-FMS-3000:Perfect_0402" H 800 1050 50  0001 C CNN
+F 2 "CJ4-MFD-Menu-Panel:Perfect_0402" H 800 1050 50  0001 C CNN
 F 3 "~" H 800 1050 50  0001 C CNN
 F 4 "0402" H 800 1050 50  0001 C CNN "JLC"
-F 5 "C15525" H 800 1050 50  0001 C CNN "LCSC"
+F 5 "" H 800 1050 50  0001 C CNN "LCSC"
 	1    800  1050
 	1    0    0    -1
@@
 F 0 "C22" H 792 2296 50  0000 L CNN
 F 1 "1uF" H 792 2205 50  0000 L CNN
-F 2 "Collins-FMS-3000:Perfect_0402" H 700 2250 50  0001 C CNN
+F 2 "CJ4-MFD-Menu-Panel:Perfect_0402" H 700 2250 50  0001 C CNN
 F 3 "~" H 700 2250 50  0001 C CNN
 F 4 "0402" H 700 2250 50  0001 C CNN "JLC"
-F 5 "C52923" H 700 2250 50  0001 C CNN "LCSC"
+F 5 "" H 700 2250 50  0001 C CNN "LCSC"
 	1    700  2250
 	1    0    0    -1
@@
 F 0 "C25" H 992 2996 50  0000 L CNN
 F 1 "1uF" H 992 2905 50  0000 L CNN
-F 2 "Collins-FMS-3000:Perfect_0402" H 900 2950 50  0001 C CNN
+F 2 "CJ4-MFD-Menu-Panel:Perfect_0402" H 900 2950 50  0001 C CNN
 F 3 "~" H 900 2950 50  0001 C CNN
 F 4 "0402" H 900 2950 50  0001 C CNN "JLC"
-F 5 "C52923" H 900 2950 50  0001 C CNN "LCSC"
+F 5 "" H 900 2950 50  0001 C CNN "LCSC"
 	1    900  2950
 	1    0    0    -1
@@
 F 0 "R21" V 2354 3650 50  0000 C CNN
 F 1 "10k" V 2445 3650 50  0000 C CNN
-F 2 "Collins-FMS-3000:Perfect_0402" H 2550 3650 50  0001 C CNN
+F 2 "CJ4-MFD-Menu-Panel:Perfect_0402" H 2550 3650 50  0001 C CNN
 F 3 "~" H 2550 3650 50  0001 C CNN
 F 4 "0402" H 2550 3650 50  0001 C CNN "JLC"
@@
 F 0 "C17" H 2392 1096 50  0000 L CNN
 F 1 "100nf" H 2392 1005 50  0000 L CNN
-F 2 "Collins-FMS-3000:Perfect_0402" H 2300 1050 50  0001 C CNN
+F 2 "CJ4-MFD-Menu-Panel:Perfect_0402" H 2300 1050 50  0001 C CNN
 F 3 "~" H 2300 1050 50  0001 C CNN
 F 4 "0402" H 2300 1050 50  0001 C CNN "JLC"
-F 5 "C1525" H 2300 1050 50  0001 C CNN "LCSC"
+F 5 "" H 2300 1050 50  0001 C CNN "LCSC"
 	1    2300 1050
 	1    0    0    -1
@@
 F 0 "C18" H 2792 1096 50  0000 L CNN
 F 1 "100nf" H 2792 1005 50  0000 L CNN
-F 2 "Collins-FMS-3000:Perfect_0402" H 2700 1050 50  0001 C CNN
+F 2 "CJ4-MFD-Menu-Panel:Perfect_0402" H 2700 1050 50  0001 C CNN
 F 3 "~" H 2700 1050 50  0001 C CNN
 F 4 "0402" H 2700 1050 50  0001 C CNN "JLC"
-F 5 "C1525" H 2700 1050 50  0001 C CNN "LCSC"
+F 5 "" H 2700 1050 50  0001 C CNN "LCSC"
 	1    2700 1050
 	1    0    0    -1
@@
 F 0 "C19" H 3192 1096 50  0000 L CNN
 F 1 "100nf" H 3192 1005 50  0000 L CNN
-F 2 "Collins-FMS-3000:Perfect_0402" H 3100 1050 50  0001 C CNN
+F 2 "CJ4-MFD-Menu-Panel:Perfect_0402" H 3100 1050 50  0001 C CNN
 F 3 "~" H 3100 1050 50  0001 C CNN
 F 4 "0402" H 3100 1050 50  0001 C CNN "JLC"
-F 5 "C1525" H 3100 1050 50  0001 C CNN "LCSC"
+F 5 "" H 3100 1050 50  0001 C CNN "LCSC"
 	1    3100 1050
 	1    0    0    -1
@@
 F 0 "C20" H 3592 1096 50  0000 L CNN
 F 1 "100nf" H 3592 1005 50  0000 L CNN
-F 2 "Collins-FMS-3000:Perfect_0402" H 3500 1050 50  0001 C CNN
+F 2 "CJ4-MFD-Menu-Panel:Perfect_0402" H 3500 1050 50  0001 C CNN
 F 3 "~" H 3500 1050 50  0001 C CNN
 F 4 "0402" H 3500 1050 50  0001 C CNN "JLC"
-F 5 "C1525" H 3500 1050 50  0001 C CNN "LCSC"
+F 5 "" H 3500 1050 50  0001 C CNN "LCSC"
 	1    3500 1050
 	1    0    0    -1
@@
 F 0 "J1" H 4307 1717 50  0000 C CNN
 F 1 "USB_B_Mini" H 4307 1626 50  0000 C CNN
-F 2 "Collins-FMS-3000:USB_B_Mini_Amphenol_UE25BE5510H" H 4400 1200 50  0001 C CNN
+F 2 "CJ4-MFD-Menu-Panel:USB_B_Mini_Amphenol_UE25BE5510H" H 4400 1200 50  0001 C CNN
 F 3 "~" H 4400 1200 50  0001 C CNN
 	1    4250 1250
@@
 F 3 "~" H 4950 1050 50  0001 C CNN
 F 4 "0805" H 4950 1050 50  0001 C CNN "JLC"
-F 5 "C72043" H 4950 1050 50  0001 C CNN "LCSC"
+F 5 "C1017" H 4950 1050 50  0001 C CNN "LCSC"
 	1    4950 1050
 	0    1    1    0
@@
 F 0 "R12" V 4754 1400 50  0000 C CNN
 F 1 "22" V 4845 1400 50  0000 C CNN
-F 2 "Collins-FMS-3000:Perfect_0402" H 4950 1400 50  0001 C CNN
+F 2 "CJ4-MFD-Menu-Panel:Perfect_0402" H 4950 1400 50  0001 C CNN
 F 3 "~" H 4950 1400 50  0001 C CNN
 F 4 "0402" H 4950 1400 50  0001 C CNN "JLC"
-F 5 "0402" H 4950 1400 50  0001 C CNN "LCSC"
+F 5 "C25092" H 4950 1400 50  0001 C CNN "LCSC"
 	1    4950 1400
 	0    1    1    0
@@
 F 0 "R14" V 4754 1700 50  0000 C CNN
 F 1 "22" V 4845 1700 50  0000 C CNN
-F 2 "Collins-FMS-3000:Perfect_0402" H 4950 1700 50  0001 C CNN
+F 2 "CJ4-MFD-Menu-Panel:Perfect_0402" H 4950 1700 50  0001 C CNN
 F 3 "~" H 4950 1700 50  0001 C CNN
 F 4 "0402" H 4950 1700 50  0001 C CNN "JLC"
-F 5 "0402" H 4950 1700 50  0001 C CNN "LCSC"
+F 5 "C25092" H 4950 1700 50  0001 C CNN "LCSC"
 	1    4950 1700
 	0    1    1    0
@@
 F 0 "C21" H 5542 1196 50  0000 L CNN
 F 1 "10uF" H 5542 1105 50  0000 L CNN
-F 2 "Collins-FMS-3000:Perfect_0402" H 5450 1150 50  0001 C CNN
+F 2 "CJ4-MFD-Menu-Panel:Perfect_0402" H 5450 1150 50  0001 C CNN
 F 3 "~" H 5450 1150 50  0001 C CNN
 F 4 "0402" H 5450 1150 50  0001 C CNN "JLC"
-F 5 "C15525" H 5450 1150 50  0001 C CNN "LCSC"
+F 5 "" H 5450 1150 50  0001 C CNN "LCSC"
 	1    5450 1150
 	1    0    0    -1
@@
 F 0 "R11" H 5959 1196 50  0000 L CNN
 F 1 "1K" H 5959 1105 50  0000 L CNN
-F 2 "Collins-FMS-3000:Perfect_0402" H 5900 1150 50  0001 C CNN
+F 2 "CJ4-MFD-Menu-Panel:Perfect_0402" H 5900 1150 50  0001 C CNN
 F 3 "~" H 5900 1150 50  0001 C CNN
 F 4 "0402" H 5900 1150 50  0001 C CNN "JLC"
@@
 F 0 "D1" V 5946 1280 50  0000 R CNN
 F 1 "GREEN" V 5855 1280 50  0000 R CNN
-F 2 "Collins-FMS-3000:LED_0603_1608Metric" V 5900 1350 50  0001 C CNN
+F 2 "LED_SMD:LED_0805_2012Metric_Pad1.15x1.40mm_HandSolder" V 5900 1350 50  0001 C CNN
 F 3 "~" V 5900 1350 50  0001 C CNN
-F 4 "0603" H 5900 1350 50  0001 C CNN "JLC"
+F 4 "" H 5900 1350 50  0001 C CNN "JLC"
 	1    5900 1350
 	0    -1   -1   0
@@
 F 0 "C26" V 4071 4500 50  0000 C CNN
 F 1 "20pF" V 4162 4500 50  0000 C CNN
-F 2 "Collins-FMS-3000:Perfect_0402" H 4300 4500 50  0001 C CNN
+F 2 "CJ4-MFD-Menu-Panel:Perfect_0402" H 4300 4500 50  0001 C CNN
 F 3 "~" H 4300 4500 50  0001 C CNN
 F 4 "0402" H 4300 4500 50  0001 C CNN "JLC"
-F 5 "C1554" H 4300 4500 50  0001 C CNN "LCSC"
+F 5 "" H 4300 4500 50  0001 C CNN "LCSC"
 	1    4300 4500
 	0    1    1    0
@@
 F 0 "C27" V 4071 5000 50  0000 C CNN
 F 1 "20pF" V 4162 5000 50  0000 C CNN
-F 2 "Collins-FMS-3000:Perfect_0402" H 4300 5000 50  0001 C CNN
+F 2 "CJ4-MFD-Menu-Panel:Perfect_0402" H 4300 5000 50  0001 C CNN
 F 3 "~" H 4300 5000 50  0001 C CNN
 F 4 "0402" H 4300 5000 50  0001 C CNN "JLC"
-F 5 "C1554" H 4300 5000 50  0001 C CNN "LCSC"
+F 5 "" H 4300 5000 50  0001 C CNN "LCSC"
 	1    4300 5000
 	0    1    1    0
@@
 F 0 "C24" H 6742 2646 50  0000 L CNN
 F 1 "100nf" H 6742 2555 50  0000 L CNN
-F 2 "Collins-FMS-3000:Perfect_0402" H 6650 2600 50  0001 C CNN
+F 2 "CJ4-MFD-Menu-Panel:Perfect_0402" H 6650 2600 50  0001 C CNN
 F 3 "~" H 6650 2600 50  0001 C CNN
 F 4 "0402" H 6650 2600 50  0001 C CNN "JLC"
-F 5 "C1525" H 6650 2600 50  0001 C CNN "LCSC"
+F 5 "" H 6650 2600 50  0001 C CNN "LCSC"
 	1    6650 2600
 	1    0    0    -1
@@
 F 0 "C23" H 6342 2646 50  0000 L CNN
 F 1 "100nf" H 6342 2555 50  0000 L CNN
-F 2 "Collins-FMS-3000:Perfect_0402" H 6250 2600 50  0001 C CNN
+F 2 "CJ4-MFD-Menu-Panel:Perfect_0402" H 6250 2600 50  0001 C CNN
 F 3 "~" H 6250 2600 50  0001 C CNN
 F 4 "0402" H 6250 2600 50  0001 C CNN "JLC"
-F 5 "C1525" H 6250 2600 50  0001 C CNN "LCSC"
+F 5 "" H 6250 2600 50  0001 C CNN "LCSC"
 	1    6250 2600
 	1    0    0    -1
@@
 F 0 "R15" H 5909 2646 50  0000 L CNN
 F 1 "10k" H 5909 2555 50  0000 L CNN
-F 2 "Collins-FMS-3000:Perfect_0402" H 5850 2600 50  0001 C CNN
+F 2 "CJ4-MFD-Menu-Panel:Perfect_0402" H 5850 2600 50  0001 C CNN
 F 3 "~" H 5850 2600 50  0001 C CNN
 F 4 "0402" H 5850 2600 50  0001 C CNN "JLC"
@@
 F 0 "R19" H 3209 3346 50  0000 L CNN
 F 1 "100k" H 3209 3255 50  0000 L CNN
-F 2 "Collins-FMS-3000:Perfect_0402" H 3150 3300 50  0001 C CNN
+F 2 "CJ4-MFD-Menu-Panel:Perfect_0402" H 3150 3300 50  0001 C CNN
 F 3 "~" H 3150 3300 50  0001 C CNN
 F 4 "0402" H 3150 3300 50  0001 C CNN "JLC"
@@
 Text HLabel 2400 4450 2    50   Input ~ 0
 CTR
-Text HLabel 2400 4350 2    50   Input ~ 0
+Text HLabel 2400 4150 2    50   Input ~ 0
 UP
 Text HLabel 2400 4250 2    50   Input ~ 0
 RIGHT
-Text HLabel 2400 4150 2    50   Input ~ 0
+Text HLabel 2400 4350 2    50   Input ~ 0
 DOWN
 Text HLabel 2400 4050 2    50   Input ~ 0

Commit message: Fix JLCPCB part assignment
Parts:
- C16, C21: LCSC (none) -> C15525
- C17, C18, C19, C20, C23, C24: LCSC (none) -> C1525
- C22, C25: LCSC (none) -> C52923
- C26, C27: LCSC (none) -> C1554
Changed lines of the file:
@@
 F 3 "~" H 800 1050 50  0001 C CNN
 F 4 "0402" H 800 1050 50  0001 C CNN "JLC"
-F 5 "" H 800 1050 50  0001 C CNN "LCSC"
+F 5 "C15525" H 800 1050 50  0001 C CNN "LCSC"
 	1    800  1050
 	1    0    0    -1
@@
 F 3 "~" H 700 2250 50  0001 C CNN
 F 4 "0402" H 700 2250 50  0001 C CNN "JLC"
-F 5 "" H 700 2250 50  0001 C CNN "LCSC"
+F 5 "C52923" H 700 2250 50  0001 C CNN "LCSC"
 	1    700  2250
 	1    0    0    -1
@@
 F 3 "~" H 900 2950 50  0001 C CNN
 F 4 "0402" H 900 2950 50  0001 C CNN "JLC"
-F 5 "" H 900 2950 50  0001 C CNN "LCSC"
+F 5 "C52923" H 900 2950 50  0001 C CNN "LCSC"
 	1    900  2950
 	1    0    0    -1
@@
 F 3 "~" H 2300 1050 50  0001 C CNN
 F 4 "0402" H 2300 1050 50  0001 C CNN "JLC"
-F 5 "" H 2300 1050 50  0001 C CNN "LCSC"
+F 5 "C1525" H 2300 1050 50  0001 C CNN "LCSC"
 	1    2300 1050
 	1    0    0    -1
@@
 F 3 "~" H 2700 1050 50  0001 C CNN
 F 4 "0402" H 2700 1050 50  0001 C CNN "JLC"
-F 5 "" H 2700 1050 50  0001 C CNN "LCSC"
+F 5 "C1525" H 2700 1050 50  0001 C CNN "LCSC"
 	1    2700 1050
 	1    0    0    -1
@@
 F 3 "~" H 3100 1050 50  0001 C CNN
 F 4 "0402" H 3100 1050 50  0001 C CNN "JLC"
-F 5 "" H 3100 1050 50  0001 C CNN "LCSC"
+F 5 "C1525" H 3100 1050 50  0001 C CNN "LCSC"
 	1    3100 1050
 	1    0    0    -1
@@
 F 3 "~" H 3500 1050 50  0001 C CNN
 F 4 "0402" H 3500 1050 50  0001 C CNN "JLC"
-F 5 "" H 3500 1050 50  0001 C CNN "LCSC"
+F 5 "C1525" H 3500 1050 50  0001 C CNN "LCSC"
 	1    3500 1050
 	1    0    0    -1
@@
 F 3 "~" H 5450 1150 50  0001 C CNN
 F 4 "0402" H 5450 1150 50  0001 C CNN "JLC"
-F 5 "" H 5450 1150 50  0001 C CNN "LCSC"
+F 5 "C15525" H 5450 1150 50  0001 C CNN "LCSC"
 	1    5450 1150
 	1    0    0    -1
@@
 F 3 "~" H 4300 4500 50  0001 C CNN
 F 4 "0402" H 4300 4500 50  0001 C CNN "JLC"
-F 5 "" H 4300 4500 50  0001 C CNN "LCSC"
+F 5 "C1554" H 4300 4500 50  0001 C CNN "LCSC"
 	1    4300 4500
 	0    1    1    0
@@
 F 3 "~" H 4300 5000 50  0001 C CNN
 F 4 "0402" H 4300 5000 50  0001 C CNN "JLC"
-F 5 "" H 4300 5000 50  0001 C CNN "LCSC"
+F 5 "C1554" H 4300 5000 50  0001 C CNN "LCSC"
 	1    4300 5000
 	0    1    1    0
@@
 F 3 "~" H 6650 2600 50  0001 C CNN
 F 4 "0402" H 6650 2600 50  0001 C CNN "JLC"
-F 5 "" H 6650 2600 50  0001 C CNN "LCSC"
+F 5 "C1525" H 6650 2600 50  0001 C CNN "LCSC"
 	1    6650 2600
 	1    0    0    -1
@@
 F 3 "~" H 6250 2600 50  0001 C CNN
 F 4 "0402" H 6250 2600 50  0001 C CNN "JLC"
-F 5 "" H 6250 2600 50  0001 C CNN "LCSC"
+F 5 "C1525" H 6250 2600 50  0001 C CNN "LCSC"
 	1    6250 2600
 	1    0    0    -1

Commit message: Ready for round two
Parts:
- D1, J1, J2, U4: JLC (none) -> DNP
Changed lines of the file:
@@
 F 2 "CJ4-MFD-Menu-Panel:USB_B_Mini_Amphenol_UE25BE5510H" H 4400 1200 50  0001 C CNN
 F 3 "~" H 4400 1200 50  0001 C CNN
+F 4 "DNP" H 4250 1250 50  0001 C CNN "JLC"
 	1    4250 1250
 	1    0    0    -1
@@
 F 2 "LED_SMD:LED_0805_2012Metric_Pad1.15x1.40mm_HandSolder" V 5900 1350 50  0001 C CNN
 F 3 "~" V 5900 1350 50  0001 C CNN
-F 4 "" H 5900 1350 50  0001 C CNN "JLC"
+F 4 "DNP" H 5900 1350 50  0001 C CNN "JLC"
 	1    5900 1350
 	0    -1   -1   0
@@
 F 2 "Connector:Tag-Connect_TC2030-IDC-NL_2x03_P1.27mm_Vertical" V 4550 2950 50  0001 C CNN
 F 3 " ~" H 3525 2350 50  0001 C CNN
+F 4 "DNP" H 4800 2900 50  0001 C CNN "JLC"
 	1    4800 2900
 	1    0    0    -1
@@
 F 2 "Package_DFN_QFN:QFN-44-1EP_7x7mm_P0.5mm_EP5.2x5.2mm" H 1800 800 50  0001 C CIN
 F 3 "http://ww1.microchip.com/downloads/en/DeviceDoc/Atmel-7766-8-bit-AVR-ATmega16U4-32U4_Datasheet.pdf" H 1800 3050 50  0001 C CNN
+F 4 "DNP" H 1800 3050 50  0001 C CNN "JLC"
 	1    1800 3050
 	1    0    0    -1
