File: CJ4-MFD-Menu-Panel.sch (KiCad schematic (older format))
At the start: 49 parts, among them SW1 SW_Push_LED, SW10 5_Way_Switch, SW11 SW_Push_LED, SW12 SW_Push_LED, SW13 SW_Push_LED, SW14 SW_Push_LED, SW15 SW_Push_LED, SW16 SW_Push_LED, SW17 SW_Push_LED, SW18 SW_Push_LED, SW19 SW_Push_LED, SW2 SW_Push_LED, SW20 SW_Push_LED, SW21 SW_Push_LED, SW3 SW_Push_LED, SW4 SW_Push_LED, SW5 SW_Push_LED, SW6 SW_Push_LED, SW7 SW_Push_LED, SW8 SW_Push_LED, SW9 SW_Push_LED, U1 MCP23017_SO, U2 MCP23017_SO, U3 IS31FL3733B

Commit message: Fix JLCPCB part assignment
Parts:
- C10, C12, C14, C6, C8: LCSC (none) -> C1525
- C11, C13, C15, C9: LCSC (none) -> C47339
- C5, C7: LCSC (none) -> C52923
Changed lines of the file:
@@
 F 3 "~" H 1050 4750 50  0001 C CNN
 F 4 "0402" H 1050 4750 50  0001 C CNN "JLC"
+F 5 "C1525" H 1050 4750 50  0001 C CNN "LCSC"
 	1    1050 4750
 	1    0    0    -1
@@
 F 3 "~" H 700 4750 50  0001 C CNN
 F 4 "0402" H 700 4750 50  0001 C CNN "JLC"
+F 5 "C52923" H 700 4750 50  0001 C CNN "LCSC"
 	1    700  4750
 	1    0    0    -1
@@
 F 3 "~" H 3750 4750 50  0001 C CNN
 F 4 "0402" H 3750 4750 50  0001 C CNN "JLC"
+F 5 "C1525" H 3750 4750 50  0001 C CNN "LCSC"
 	1    3750 4750
 	1    0    0    -1
@@
 F 3 "~" H 3400 4750 50  0001 C CNN
 F 4 "0402" H 3400 4750 50  0001 C CNN "JLC"
+F 5 "C52923" H 3400 4750 50  0001 C CNN "LCSC"
 	1    3400 4750
 	1    0    0    -1
@@
 F 3 "~" H 9050 4850 50  0001 C CNN
 F 4 "0402" H 9050 4850 50  0001 C CNN "JLC"
+F 5 "C47339" H 9050 4850 50  0001 C CNN "LCSC"
 	1    9050 4850
 	1    0    0    -1
@@
 F 3 "~" H 9050 2900 50  0001 C CNN
 F 4 "0402" H 9050 2900 50  0001 C CNN "JLC"
+F 5 "C1525" H 9050 2900 50  0001 C CNN "LCSC"
 	1    9050 2900
 	1    0    0    -1
@@
 F 3 "~" H 8600 2900 50  0001 C CNN
 F 4 "0402" H 8600 2900 50  0001 C CNN "JLC"
+F 5 "C47339" H 8600 2900 50  0001 C CNN "LCSC"
 	1    8600 2900
 	1    0    0    -1
@@
 F 3 "~" H 9050 3200 50  0001 C CNN
 F 4 "0402" H 9050 3200 50  0001 C CNN "JLC"
+F 5 "C1525" H 9050 3200 50  0001 C CNN "LCSC"
 	1    9050 3200
 	1    0    0    -1
@@
 F 3 "~" H 8600 3200 50  0001 C CNN
 F 4 "0402" H 8600 3200 50  0001 C CNN "JLC"
+F 5 "C47339" H 8600 3200 50  0001 C CNN "LCSC"
 	1    8600 3200
 	1    0    0    -1
@@
 F 3 "~" H 9050 3550 50  0001 C CNN
 F 4 "0402" H 9050 3550 50  0001 C CNN "JLC"
+F 5 "C1525" H 9050 3550 50  0001 C CNN "LCSC"
 	1    9050 3550
 	1    0    0    -1
@@
 F 3 "~" H 8600 3550 50  0001 C CNN
 F 4 "0402" H 8600 3550 50  0001 C CNN "JLC"
+F 5 "C47339" H 8600 3550 50  0001 C CNN "LCSC"
 	1    8600 3550
 	1    0    0    -1

Commit message: Ready for round two
Parts:
- ENC1, H1, H2, H3, H4, H5, H6, H7, SW1, SW10, SW11, SW12, SW13, SW14, SW15, SW16, SW17, SW18, SW19, SW2, SW20, SW21, SW3, SW4, SW5, SW6, SW7, SW8, SW9, U1, U2, U3: JLC (none) -> DNP
Changed lines of the file:
@@
 F 2 "CJ4-MFD-Menu-Panel:SW_PUSH_6mm" H 3850 600 50  0001 C CNN
 F 3 "" H 3850 600 50  0001 C CNN
+F 4 "DNP" H 3850 600 50  0001 C CNN "JLC"
 	1    3850 600
 	1    0    0    -1
@@
 F 2 "CJ4-MFD-Menu-Panel:SW_PUSH_6mm" H 4900 600 50  0001 C CNN
 F 3 "" H 4900 600 50  0001 C CNN
+F 4 "DNP" H 4900 600 50  0001 C CNN "JLC"
 	1    4900 600
 	1    0    0    -1
@@
 F 2 "CJ4-MFD-Menu-Panel:SW_PUSH_6mm" H 6000 600 50  0001 C CNN
 F 3 "" H 6000 600 50  0001 C CNN
+F 4 "DNP" H 6000 600 50  0001 C CNN "JLC"
 	1    6000 600
 	1    0    0    -1
@@
 F 2 "CJ4-MFD-Menu-Panel:SW_PUSH_6mm" H 850 950 50  0001 C CNN
 F 3 "" H 850 950 50  0001 C CNN
+F 4 "DNP" H 850 950 50  0001 C CNN "JLC"
 	1    850  950
 	1    0    0    -1
@@
 F 2 "CJ4-MFD-Menu-Panel:SW_PUSH_6mm" H 850 1300 50  0001 C CNN
 F 3 "" H 850 1300 50  0001 C CNN
+F 4 "DNP" H 850 1300 50  0001 C CNN "JLC"
 	1    850  1300
 	1    0    0    -1
@@
 F 2 "CJ4-MFD-Menu-Panel:SW_PUSH_6mm" H 850 1650 50  0001 C CNN
 F 3 "" H 850 1650 50  0001 C CNN
+F 4 "DNP" H 850 1650 50  0001 C CNN "JLC"
 	1    850  1650
 	1    0    0    -1
@@
 F 2 "CJ4-MFD-Menu-Panel:SW_PUSH_6mm" H 1900 1650 50  0001 C CNN
 F 3 "" H 1900 1650 50  0001 C CNN
+F 4 "DNP" H 1900 1650 50  0001 C CNN "JLC"
 	1    1900 1650
 	1    0    0    -1
@@
 F 2 "CJ4-MFD-Menu-Panel:SW_PUSH_6mm" H 2850 1650 50  0001 C CNN
 F 3 "" H 2850 1650 50  0001 C CNN
+F 4 "DNP" H 2850 1650 50  0001 C CNN "JLC"
 	1    2850 1650
 	1    0    0    -1
@@
 F 2 "CJ4-MFD-Menu-Panel:SW_PUSH_6mm" H 3850 1650 50  0001 C CNN
 F 3 "" H 3850 1650 50  0001 C CNN
+F 4 "DNP" H 3850 1650 50  0001 C CNN "JLC"
 	1    3850 1650
 	1    0    0    -1
@@
 F 2 "CJ4-MFD-Menu-Panel:SW_PUSH_6mm" H 4900 1650 50  0001 C CNN
 F 3 "" H 4900 1650 50  0001 C CNN
+F 4 "DNP" H 4900 1650 50  0001 C CNN "JLC"
 	1    4900 1650
 	1    0    0    -1
@@
 F 2 "CJ4-MFD-Menu-Panel:SW_PUSH_6mm" H 6000 1650 50  0001 C CNN
 F 3 "" H 6000 1650 50  0001 C CNN
+F 4 "DNP" H 6000 1650 50  0001 C CNN "JLC"
 	1    6000 1650
 	1    0    0    -1
@@
 F 2 "CJ4-MFD-Menu-Panel:SW_PUSH_6mm" H 7050 1650 50  0001 C CNN
 F 3 "" H 7050 1650 50  0001 C CNN
+F 4 "DNP" H 7050 1650 50  0001 C CNN "JLC"
 	1    7050 1650
 	1    0    0    -1
@@
 F 2 "CJ4-MFD-Menu-Panel:SW_PUSH_6mm" H 3850 950 50  0001 C CNN
 F 3 "" H 3850 950 50  0001 C CNN
+F 4 "DNP" H 3850 950 50  0001 C CNN "JLC"
 	1    3850 950
 	1    0    0    -1
@@
 F 2 "CJ4-MFD-Menu-Panel:SW_PUSH_6mm" H 3850 1300 50  0001 C CNN
 F 3 "" H 3850 1300 50  0001 C CNN
+F 4 "DNP" H 3850 1300 50  0001 C CNN "JLC"
 	1    3850 1300
 	1    0    0    -1
@@
 F 2 "CJ4-MFD-Menu-Panel:SW_PUSH_6mm" H 4900 950 50  0001 C CNN
 F 3 "" H 4900 950 50  0001 C CNN
+F 4 "DNP" H 4900 950 50  0001 C CNN "JLC"
 	1    4900 950
 	1    0    0    -1
@@
 F 2 "CJ4-MFD-Menu-Panel:SW_PUSH_6mm" H 4900 1300 50  0001 C CNN
 F 3 "" H 4900 1300 50  0001 C CNN
+F 4 "DNP" H 4900 1300 50  0001 C CNN "JLC"
 	1    4900 1300
 	1    0    0    -1
@@
 F 2 "CJ4-MFD-Menu-Panel:SW_PUSH_6mm" H 6000 1300 50  0001 C CNN
 F 3 "" H 6000 1300 50  0001 C CNN
+F 4 "DNP" H 6000 1300 50  0001 C CNN "JLC"
 	1    6000 1300
 	1    0    0    -1
@@
 F 2 "CJ4-MFD-Menu-Panel:SW_PUSH_6mm" H 2850 600 50  0001 C CNN
 F 3 "" H 2850 600 50  0001 C CNN
+F 4 "DNP" H 2850 600 50  0001 C CNN "JLC"
 	1    2850 600
 	1    0    0    -1
@@
 F 2 "CJ4-MFD-Menu-Panel:SW_PUSH_6mm" H 1900 600 50  0001 C CNN
 F 3 "" H 1900 600 50  0001 C CNN
+F 4 "DNP" H 1900 600 50  0001 C CNN "JLC"
 	1    1900 600
 	1    0    0    -1
@@
 F 2 "CJ4-MFD-Menu-Panel:SW_PUSH_6mm" H 850 600 50  0001 C CNN
 F 3 "" H 850 600 50  0001 C CNN
+F 4 "DNP" H 850 600 50  0001 C CNN "JLC"
 	1    850  600
 	1    0    0    -1
@@
 F 2 "CJ4-MFD-Menu-Panel:5_Way_Switch" H 8650 1150 50  0001 C CNN
 F 3 "" H 8650 1150 50  0001 C CNN
+F 4 "DNP" H 8650 1150 50  0001 C CNN "JLC"
 	1    8650 1150
 	1    0    0    -1
@@
 F 2 "CJ4-MFD-Menu-Panel:SW_PUSH_6mm" H 4550 2300 50  0001 C CNN
 F 3 "" H 4550 2300 50  0001 C CNN
+F 4 "DNP" H 4550 2300 50  0001 C CNN "JLC"
 	2    4550 2300
 	1    0    0    -1
@@
 F 2 "CJ4-MFD-Menu-Panel:SW_PUSH_6mm" H 4950 2300 50  0001 C CNN
 F 3 "" H 4950 2300 50  0001 C CNN
+F 4 "DNP" H 4950 2300 50  0001 C CNN "JLC"
 	2    4950 2300
 	1    0    0    -1
@@
 F 2 "CJ4-MFD-Menu-Panel:SW_PUSH_6mm" H 5350 2300 50  0001 C CNN
 F 3 "" H 5350 2300 50  0001 C CNN
+F 4 "DNP" H 5350 2300 50  0001 C CNN "JLC"
 	2    5350 2300
 	1    0    0    -1
@@
 F 2 "CJ4-MFD-Menu-Panel:SW_PUSH_6mm" H 5750 2300 50  0001 C CNN
 F 3 "" H 5750 2300 50  0001 C CNN
+F 4 "DNP" H 5750 2300 50  0001 C CNN "JLC"
 	2    5750 2300
 	1    0    0    -1
@@
 F 2 "CJ4-MFD-Menu-Panel:SW_PUSH_6mm" H 6150 2300 50  0001 C CNN
 F 3 "" H 6150 2300 50  0001 C CNN
+F 4 "DNP" H 6150 2300 50  0001 C CNN "JLC"
 	2    6150 2300
 	1    0    0    -1
@@
 F 2 "CJ4-MFD-Menu-Panel:SW_PUSH_6mm" H 6550 2300 50  0001 C CNN
 F 3 "" H 6550 2300 50  0001 C CNN
+F 4 "DNP" H 6550 2300 50  0001 C CNN "JLC"
 	2    6550 2300
 	1    0    0    -1
@@
 F 2 "CJ4-MFD-Menu-Panel:SW_PUSH_6mm" H 4550 2650 50  0001 C CNN
 F 3 "" H 4550 2650 50  0001 C CNN
+F 4 "DNP" H 4550 2650 50  0001 C CNN "JLC"
 	2    4550 2650
 	1    0    0    -1
@@
 F 2 "CJ4-MFD-Menu-Panel:SW_PUSH_6mm" H 4550 3000 50  0001 C CNN
 F 3 "" H 4550 3000 50  0001 C CNN
+F 4 "DNP" H 4550 3000 50  0001 C CNN "JLC"
 	2    4550 3000
 	1    0    0    -1
@@
 F 2 "CJ4-MFD-Menu-Panel:SW_PUSH_6mm" H 4550 3350 50  0001 C CNN
 F 3 "" H 4550 3350 50  0001 C CNN
+F 4 "DNP" H 4550 3350 50  0001 C CNN "JLC"
 	2    4550 3350
 	1    0    0    -1
@@
 F 2 "CJ4-MFD-Menu-Panel:SW_PUSH_6mm" H 4950 3350 50  0001 C CNN
 F 3 "" H 4950 3350 50  0001 C CNN
+F 4 "DNP" H 4950 3350 50  0001 C CNN "JLC"
 	2    4950 3350
 	1    0    0    -1
@@
 F 2 "CJ4-MFD-Menu-Panel:SW_PUSH_6mm" H 5350 3350 50  0001 C CNN
 F 3 "" H 5350 3350 50  0001 C CNN
+F 4 "DNP" H 5350 3350 50  0001 C CNN "JLC"
 	2    5350 3350
 	1    0    0    -1
@@
 F 2 "CJ4-MFD-Menu-Panel:SW_PUSH_6mm" H 5750 3350 50  0001 C CNN
 F 3 "" H 5750 3350 50  0001 C CNN
+F 4 "DNP" H 5750 3350 50  0001 C CNN "JLC"
 	2    5750 3350
 	1    0    0    -1
@@
 F 2 "CJ4-MFD-Menu-Panel:SW_PUSH_6mm" H 6150 3350 50  0001 C CNN
 F 3 "" H 6150 3350 50  0001 C CNN
+F 4 "DNP" H 6150 3350 50  0001 C CNN "JLC"
 	2    6150 3350
 	1    0    0    -1
@@
 F 2 "CJ4-MFD-Menu-Panel:SW_PUSH_6mm" H 6550 3350 50  0001 C CNN
 F 3 "" H 6550 3350 50  0001 C CNN
+F 4 "DNP" H 6550 3350 50  0001 C CNN "JLC"
 	2    6550 3350
 	1    0    0    -1
@@
 F 2 "CJ4-MFD-Menu-Panel:SW_PUSH_6mm" H 6950 3350 50  0001 C CNN
 F 3 "" H 6950 3350 50  0001 C CNN
+F 4 "DNP" H 6950 3350 50  0001 C CNN "JLC"
 	2    6950 3350
 	1    0    0    -1
@@
 F 2 "CJ4-MFD-Menu-Panel:SW_PUSH_6mm" H 6550 3000 50  0001 C CNN
 F 3 "" H 6550 3000 50  0001 C CNN
+F 4 "DNP" H 6550 3000 50  0001 C CNN "JLC"
 	2    6550 3000
 	1    0    0    -1
@@
 F 2 "CJ4-MFD-Menu-Panel:SW_PUSH_6mm" H 6150 3000 50  0001 C CNN
 F 3 "" H 6150 3000 50  0001 C CNN
+F 4 "DNP" H 6150 3000 50  0001 C CNN "JLC"
 	2    6150 3000
 	1    0    0    -1
@@
 F 2 "CJ4-MFD-Menu-Panel:SW_PUSH_6mm" H 6150 2650 50  0001 C CNN
 F 3 "" H 6150 2650 50  0001 C CNN
+F 4 "DNP" H 6150 2650 50  0001 C CNN "JLC"
 	2    6150 2650
 	1    0    0    -1
@@
 F 2 "CJ4-MFD-Menu-Panel:SW_PUSH_6mm" H 5750 3000 50  0001 C CNN
 F 3 "" H 5750 3000 50  0001 C CNN
+F 4 "DNP" H 5750 3000 50  0001 C CNN "JLC"
 	2    5750 3000
 	1    0    0    -1
@@
 F 2 "CJ4-MFD-Menu-Panel:SW_PUSH_6mm" H 5750 2650 50  0001 C CNN
 F 3 "" H 5750 2650 50  0001 C CNN
+F 4 "DNP" H 5750 2650 50  0001 C CNN "JLC"
 	2    5750 2650
 	1    0    0    -1
@@
 F 2 "Package_QFP:TQFP-48-1EP_7x7mm_P0.5mm_EP5x5mm_ThermalVias" H 9800 1350 50  0001 C CNN
 F 3 "https://www.lumissil.com/assets/pdf/core/IS31FL3733B_DS.pdf" H 9800 3850 50  0001 C CNN
+F 4 "DNP" H 9800 3850 50  0001 C CNN "JLC"
 	1    9800 3850
 	1    0    0    -1
@@
 F 21 "+85°C" H 2600 5300 50  0001 L CNN "temperature range high"
 F 22 "-40°C" H 2600 5400 50  0001 L CNN "temperature range low"
+F 23 "DNP" H 2600 2900 50  0001 C CNN "JLC"
 	1    2600 2900
 	1    0    0    -1
@@
 F 2 "Package_SO:SOIC-28W_7.5x17.9mm_P1.27mm" H 2000 5050 50  0001 L CNN
 F 3 "http://ww1.microchip.com/downloads/en/DeviceDoc/20001952C.pdf" H 2000 4950 50  0001 L CNN
+F 4 "DNP" H 1800 6050 50  0001 C CNN "JLC"
 	1    1800 6050
 	1    0    0    -1
@@
 F 2 "Package_SO:SOIC-28W_7.5x17.9mm_P1.27mm" H 4700 5050 50  0001 L CNN
 F 3 "http://ww1.microchip.com/downloads/en/DeviceDoc/20001952C.pdf" H 4700 4950 50  0001 L CNN
+F 4 "DNP" H 4500 6050 50  0001 C CNN "JLC"
 	1    4500 6050
 	1    0    0    -1
@@
 F 2 "MountingHole:MountingHole_3.2mm_M3" H 7550 2600 50  0001 C CNN
 F 3 "~" H 7550 2600 50  0001 C CNN
+F 4 "DNP" H 7550 2600 50  0001 C CNN "JLC"
 	1    7550 2600
 	1    0    0    -1
@@
 F 2 "MountingHole:MountingHole_3.2mm_M3" H 7550 2800 50  0001 C CNN
 F 3 "~" H 7550 2800 50  0001 C CNN
+F 4 "DNP" H 7550 2800 50  0001 C CNN "JLC"
 	1    7550 2800
 	1    0    0    -1
@@
 F 2 "MountingHole:MountingHole_3.2mm_M3" H 7550 3000 50  0001 C CNN
 F 3 "~" H 7550 3000 50  0001 C CNN
+F 4 "DNP" H 7550 3000 50  0001 C CNN "JLC"
 	1    7550 3000
 	1    0    0    -1
@@
 F 2 "MountingHole:MountingHole_3.2mm_M3" H 7550 3200 50  0001 C CNN
 F 3 "~" H 7550 3200 50  0001 C CNN
+F 4 "DNP" H 7550 3200 50  0001 C CNN "JLC"
 	1    7550 3200
 	1    0    0    -1
@@
 F 2 "CJ4-MFD-Menu-Panel:JLCPCB_Tooling_Hole" H 7550 3400 50  0001 C CNN
 F 3 "~" H 7550 3400 50  0001 C CNN
+F 4 "DNP" H 7550 3400 50  0001 C CNN "JLC"
 	1    7550 3400
 	1    0    0    -1
@@
 F 2 "CJ4-MFD-Menu-Panel:JLCPCB_Tooling_Hole" H 7550 3600 50  0001 C CNN
 F 3 "~" H 7550 3600 50  0001 C CNN
+F 4 "DNP" H 7550 3600 50  0001 C CNN "JLC"
 	1    7550 3600
 	1    0    0    -1
@@
 F 2 "CJ4-MFD-Menu-Panel:JLCPCB_Tooling_Hole" H 7550 3800 50  0001 C CNN
 F 3 "~" H 7550 3800 50  0001 C CNN
+F 4 "DNP" H 7550 3800 50  0001 C CNN "JLC"
 	1    7550 3800
 	1    0    0    -1

Commit message: Rename a global label to match event name
Connections:
- net E_BTN renamed DATA
Changed lines of the file:
@@
 	3950 2900 3950 3750
 Text GLabel 3600 3000 2    50   Output ~ 0
-E_BTN
+DATA
 $Comp
 L power:+5V #PWR0101
@@
 PASS_BRIEF
 Text GLabel 2500 6150 2    50   Input ~ 0
-E_BTN
+DATA
 Text GLabel 8300 1150 0    50   Output ~ 0
 LEFT
